Commit message: add fingertip frame

File: src/assets/canonical/urdf/allegro_hand_left.urdf (robot description, URDF)
Before this commit: robot DexterousHand, 24 links, 23 joints
Links:
- added link index_tip
- added link little_tip
- added link middle_tip
- added link ring_tip
- added link thumb_tip
Joints:
- added joint index_joint_tip: type fixed, parent index_distal, child index_tip, origin xyz=0 0 0.0387 rpy=0 0 0
- added joint little_joint_tip: type fixed, parent little_distal, child little_tip, origin xyz=0 0 0.0387 rpy=0 0 0
- added joint middle_joint_tip: type fixed, parent middle_distal, child middle_tip, origin xyz=0 0 0.0387 rpy=0 0 0
- added joint ring_joint_tip: type fixed, parent ring_distal, child ring_tip, origin xyz=0 0 0.0387 rpy=0 0 0
- added joint thumb_joint_tip: type fixed, parent thumb_distal, child thumb_tip, origin xyz=0 0 0.0543 rpy=0 0 0

File: src/assets/canonical/urdf/allegro_hand_right.urdf (robot description, URDF)
Before this commit: robot DexterousHand, 24 links, 23 joints
Links:
- added link index_tip
- added link little_tip
- added link middle_tip
- added link ring_tip
- added link thumb_tip
Joints:
- added joint index_joint_tip: type fixed, parent index_distal, child index_tip, origin xyz=0 0 0.0387 rpy=0 0 0
- added joint little_joint_tip: type fixed, parent little_distal, child little_tip, origin xyz=0 0 0.0387 rpy=0 0 0
- added joint middle_joint_tip: type fixed, parent middle_distal, child middle_tip, origin xyz=0 0 0.0387 rpy=0 0 0
- added joint ring_joint_tip: type fixed, parent ring_distal, child ring_tip, origin xyz=0 0 0.0387 rpy=0 0 0
- added joint thumb_joint_tip: type fixed, parent thumb_distal, child thumb_tip, origin xyz=0 0 0.0543 rpy=0 0 0
- joint ring_joint3: origin xyz=0 0 0.054 rpy=0 0 0 -> xyz=0 0 0 rpy=0 0 0
- joint ring_joint4: origin xyz=0 0 0.0384 rpy=0 0 0 -> xyz=0 0 0 rpy=0 0 0

File: src/assets/canonical/urdf/barrett_hand.urdf (robot description, URDF)
Before this commit: robot DexterousHand, 24 links, 23 joints
Links:
- added link index_tip
- added link little_tip
- added link middle_tip
- added link ring_tip
- added link thumb_tip
Joints:
- added joint index_joint_tip: type fixed, parent index_distal, child index_tip, origin xyz=0 0 0.064 rpy=0 0 0
- added joint little_joint_tip: type fixed, parent little_distal, child little_tip, origin xyz=0 0 0.064 rpy=0 0 0
- added joint middle_joint_tip: type fixed, parent middle_distal, child middle_tip, origin xyz=0 0 0.064 rpy=0 0 0
- added joint ring_joint_tip: type fixed, parent ring_distal, child ring_tip, origin xyz=0 0 0.064 rpy=0 0 0
- added joint thumb_joint_tip: type fixed, parent thumb_distal, child thumb_tip, origin xyz=0 0 0.064 rpy=0 0 0

File: src/assets/canonical/urdf/dex3_left.urdf (robot description, URDF)
Before this commit: robot DexterousHand, 24 links, 23 joints
Links:
- added link index_tip
- added link little_tip
- added link middle_tip
- added link ring_tip
- added link thumb_tip
Joints:
- added joint index_joint_tip: type fixed, parent index_distal, child index_tip, origin xyz=0 0 0.05 rpy=0 0 0
- added joint little_joint_tip: type fixed, parent little_distal, child little_tip, origin xyz=0 0 0.05 rpy=0 0 0
- added joint middle_joint_tip: type fixed, parent middle_distal, child middle_tip, origin xyz=0 0 0.05 rpy=0 0 0
- added joint ring_joint_tip: type fixed, parent ring_distal, child ring_tip, origin xyz=0 0 0.05 rpy=0 0 0
- added joint thumb_joint_tip: type fixed, parent thumb_distal, child thumb_tip, origin xyz=0 0 0.05 rpy=0 0 0
- joint index_joint4: origin xyz=0 0 0.0 rpy=0 0 0 -> xyz=0 0 0 rpy=0 0 0
- joint little_joint3: origin xyz=0 0 0.0458 rpy=0 0 0 -> xyz=0 0 0 rpy=0 0 0
- joint little_joint4: origin xyz=0 0 0.0 rpy=0 0 0 -> xyz=0 0 0 rpy=0 0 0
- joint middle_joint4: origin xyz=0 0 0.0 rpy=0 0 0 -> xyz=0 0 0 rpy=0 0 0
- joint ring_joint3: origin xyz=0 0 0.0458 rpy=0 0 0 -> xyz=0 0 0 rpy=0 0 0
- joint ring_joint4: origin xyz=0 0 0.0 rpy=0 0 0 -> xyz=0 0 0 rpy=0 0 0
- joint thumb_joint5: origin xyz=0 0 0.0 rpy=0 0 0 -> xyz=0 0 0 rpy=0 0 0

File: src/assets/canonical/urdf/dex3_right.urdf (robot description, URDF)
Before this commit: robot DexterousHand, 24 links, 23 joints
Links:
- added link index_tip
- added link little_tip
- added link middle_tip
- added link ring_tip
- added link thumb_tip
Joints:
- added joint index_joint_tip: type fixed, parent index_distal, child index_tip, origin xyz=0 0 0.05 rpy=0 0 0
- added joint little_joint_tip: type fixed, parent little_distal, child little_tip, origin xyz=0 0 0.05 rpy=0 0 0
- added joint middle_joint_tip: type fixed, parent middle_distal, child middle_tip, origin xyz=0 0 0.05 rpy=0 0 0
- added joint ring_joint_tip: type fixed, parent ring_distal, child ring_tip, origin xyz=0 0 0.05 rpy=0 0 0
- added joint thumb_joint_tip: type fixed, parent thumb_distal, child thumb_tip, origin xyz=0 0 0.05 rpy=0 0 0
- joint index_joint4: origin xyz=0 0 0.0 rpy=0 0 0 -> xyz=0 0 0 rpy=0 0 0
- joint little_joint3: origin xyz=0 0 0.0458 rpy=0 0 0 -> xyz=0 0 0 rpy=0 0 0
- joint little_joint4: origin xyz=0 0 0.0 rpy=0 0 0 -> xyz=0 0 0 rpy=0 0 0
- joint middle_joint4: origin xyz=0 0 0.0 rpy=0 0 0 -> xyz=0 0 0 rpy=0 0 0
- joint ring_joint3: origin xyz=0 0 0.0458 rpy=0 0 0 -> xyz=0 0 0 rpy=0 0 0
- joint ring_joint4: origin xyz=0 0 0.0 rpy=0 0 0 -> xyz=0 0 0 rpy=0 0 0
- joint thumb_joint5: origin xyz=0 0 0.0 rpy=0 0 0 -> xyz=0 0 0 rpy=0 0 0

File: src/assets/canonical/urdf/gaia_hand_left.urdf (robot description, URDF)
Before this commit: robot DexterousHand, 24 links, 23 joints
Links:
- added link index_tip
- added link little_tip
- added link middle_tip
- added link ring_tip
- added link thumb_tip
- link index_distal: mass 0.013577366879999999 -> 0.014137199999999999; geometry collision cylinder length=0.024999999999999998 radius=0.01; collision sphere radius=0.01
- link index_proximal: mass 0.014361836966400001 -> 0.014954016; geometry collision cylinder length=0.027600000000000003 radius=0.01; collision sphere radius=0.01
- link little_distal: mass 0.013577366879999999 -> 0.014137199999999999; geometry collision cylinder length=0.024999999999999998 radius=0.01; collision sphere radius=0.01
- link little_proximal: mass 0.014361836966400001 -> 0.014954016; geometry collision cylinder length=0.027600000000000003 radius=0.01; collision sphere radius=0.01
- link middle_distal: mass 0.013577366879999999 -> 0.014137199999999999; geometry collision cylinder length=0.024999999999999998 radius=0.01; collision sphere radius=0.01
- link middle_proximal: mass 0.014361836966400001 -> 0.014954016; geometry collision cylinder length=0.027600000000000003 radius=0.01; collision sphere radius=0.01
- link palm: mass 0.1539384 -> 0.15708000000000003; geometry collision cylinder length=0.02 radius=0.05; visual cylinder length=0.02 radius=0.05
- link ring_distal: mass 0.013577366879999999 -> 0.014137199999999999; geometry collision cylinder length=0.024999999999999998 radius=0.01; collision sphere radius=0.01
- link ring_proximal: mass 0.014361836966400001 -> 0.014954016; geometry collision cylinder length=0.027600000000000003 radius=0.01; collision sphere radius=0.01
- link thumb_distal: mass 0.013577366879999999 -> 0.014137199999999999; geometry collision cylinder length=0.024999999999999998 radius=0.01; collision sphere radius=0.01
- link thumb_proximal: mass 0.0162626683296 -> 0.016933224; geometry collision cylinder length=0.0339 radius=0.01; collision sphere radius=0.01
Joints:
- added joint index_joint_tip: type fixed, parent index_distal, child index_tip, origin xyz=0 0 0.045 rpy=0 0 0
- added joint little_joint_tip: type fixed, parent little_distal, child little_tip, origin xyz=0 0 0.045 rpy=0 0 0
- added joint middle_joint_tip: type fixed, parent middle_distal, child middle_tip, origin xyz=0 0 0.045 rpy=0 0 0
- added joint ring_joint_tip: type fixed, parent ring_distal, child ring_tip, origin xyz=0 0 0.045 rpy=0 0 0
- added joint thumb_joint_tip: type fixed, parent thumb_distal, child thumb_tip, origin xyz=0 0 0.045 rpy=0 0 0

File: src/assets/canonical/urdf/gaia_hand_right.urdf (robot description, URDF)
Before this commit: robot DexterousHand, 24 links, 23 joints
Links:
- added link index_tip
- added link little_tip
- added link middle_tip
- added link ring_tip
- added link thumb_tip
Joints:
- added joint index_joint_tip: type fixed, parent index_distal, child index_tip, origin xyz=0 0 0.045 rpy=0 0 0
- added joint little_joint_tip: type fixed, parent little_distal, child little_tip, origin xyz=0 0 0.045 rpy=0 0 0
- added joint middle_joint_tip: type fixed, parent middle_distal, child middle_tip, origin xyz=0 0 0.045 rpy=0 0 0
- added joint ring_joint_tip: type fixed, parent ring_distal, child ring_tip, origin xyz=0 0 0.045 rpy=0 0 0
- added joint thumb_joint_tip: type fixed, parent thumb_distal, child thumb_tip, origin xyz=0 0 0.045 rpy=0 0 0

File: src/assets/canonical/urdf/leap_hand_left.urdf (robot description, URDF)
Before this commit: robot DexterousHand, 24 links, 23 joints
Links:
- added link index_tip
- added link little_tip
- added link middle_tip
- added link ring_tip
- added link thumb_tip
Joints:
- added joint index_joint_tip: type fixed, parent index_distal, child index_tip, origin xyz=0 0 0.052 rpy=0 0 0
- added joint little_joint_tip: type fixed, parent little_distal, child little_tip, origin xyz=0 0 0.052 rpy=0 0 0
- added joint middle_joint_tip: type fixed, parent middle_distal, child middle_tip, origin xyz=0 0 0.052 rpy=0 0 0
- added joint ring_joint_tip: type fixed, parent ring_distal, child ring_tip, origin xyz=0 0 0.052 rpy=0 0 0
- added joint thumb_joint_tip: type fixed, parent thumb_distal, child thumb_tip, origin xyz=0 0 0.06 rpy=0 0 0
- joint ring_joint3: origin xyz=0 0 0.0531 rpy=0 0 0 -> xyz=0 0 0 rpy=0 0 0
- joint ring_joint4: origin xyz=0 0 0.0361 rpy=0 0 0 -> xyz=0 0 0 rpy=0 0 0

File: src/assets/canonical/urdf/leap_hand_right.urdf (robot description, URDF)
Before this commit: robot DexterousHand, 24 links, 23 joints
Links:
- added link index_tip
- added link little_tip
- added link middle_tip
- added link ring_tip
- added link thumb_tip
Joints:
- added joint index_joint_tip: type fixed, parent index_distal, child index_tip, origin xyz=0 0 0.052 rpy=0 0 0
- added joint little_joint_tip: type fixed, parent little_distal, child little_tip, origin xyz=0 0 0.052 rpy=0 0 0
- added joint middle_joint_tip: type fixed, parent middle_distal, child middle_tip, origin xyz=0 0 0.052 rpy=0 0 0
- added joint ring_joint_tip: type fixed, parent ring_distal, child ring_tip, origin xyz=0 0 0.052 rpy=0 0 0
- added joint thumb_joint_tip: type fixed, parent thumb_distal, child thumb_tip, origin xyz=0 0 0.06 rpy=0 0 0
- joint ring_joint3: origin xyz=0 0 0.0531 rpy=0 0 0 -> xyz=0 0 0 rpy=0 0 0
- joint ring_joint4: origin xyz=0 0 0.0361 rpy=0 0 0 -> xyz=0 0 0 rpy=0 0 0

File: src/assets/canonical/urdf/shadow_hand_left.urdf (robot description, URDF)
Before this commit: robot DexterousHand, 24 links, 23 joints
Links:
- added link index_tip
- added link little_tip
- added link middle_tip
- added link ring_tip
- added link thumb_tip
Joints:
- added joint index_joint_tip: type fixed, parent index_distal, child index_tip, origin xyz=0 0 0.035 rpy=0 0 0
- added joint little_joint_tip: type fixed, parent little_distal, child little_tip, origin xyz=0 0 0.035 rpy=0 0 0
- added joint middle_joint_tip: type fixed, parent middle_distal, child middle_tip, origin xyz=0 0 0.035 rpy=0 0 0
- added joint ring_joint_tip: type fixed, parent ring_distal, child ring_tip, origin xyz=0 0 0.035 rpy=0 0 0
- added joint thumb_joint_tip: type fixed, parent thumb_distal, child thumb_tip, origin xyz=0 0 0.035 rpy=0 0 0

File: src/assets/canonical/urdf/shadow_hand_right.urdf (robot description, URDF)
Before this commit: robot DexterousHand, 24 links, 23 joints
Links:
- added link index_tip
- added link little_tip
- added link middle_tip
- added link ring_tip
- added link thumb_tip
Joints:
- added joint index_joint_tip: type fixed, parent index_distal, child index_tip, origin xyz=0 0 0.035 rpy=0 0 0
- added joint little_joint_tip: type fixed, parent little_distal, child little_tip, origin xyz=0 0 0.035 rpy=0 0 0
- added joint middle_joint_tip: type fixed, parent middle_distal, child middle_tip, origin xyz=0 0 0.035 rpy=0 0 0
- added joint ring_joint_tip: type fixed, parent ring_distal, child ring_tip, origin xyz=0 0 0.035 rpy=0 0 0
- added joint thumb_joint_tip: type fixed, parent thumb_distal, child thumb_tip, origin xyz=0 0 0.035 rpy=0 0 0

File: src/assets/canonical/urdf/sharpa_wave_left.urdf (robot description, URDF)
Before this commit: robot DexterousHand, 24 links, 23 joints
Links:
- added link index_tip
- added link little_tip
- added link middle_tip
- added link ring_tip
- added link thumb_tip
Joints:
- added joint index_joint_tip: type fixed, parent index_distal, child index_tip, origin xyz=0 0 0.026 rpy=0 0 0
- added joint little_joint_tip: type fixed, parent little_distal, child little_tip, origin xyz=0 0 0.026 rpy=0 0 0
- added joint middle_joint_tip: type fixed, parent middle_distal, child middle_tip, origin xyz=0 0 0.026 rpy=0 0 0
- added joint ring_joint_tip: type fixed, parent ring_distal, child ring_tip, origin xyz=0 0 0.026 rpy=0 0 0
- added joint thumb_joint_tip: type fixed, parent thumb_distal, child thumb_tip, origin xyz=0 0 0.028 rpy=0 0 0
- joint thumb_joint1: origin xyz=0.0154 -0.026 0.0129 rpy=0.46364738 -0.65906055 0.88607899 -> xyz=0.0154 -0.026 0.0129 rpy=0.4636 -0.6591 0.8861

File: src/assets/canonical/urdf/sharpa_wave_right.urdf (robot description, URDF)
Before this commit: robot DexterousHand, 24 links, 23 joints
Links:
- added link index_tip
- added link little_tip
- added link middle_tip
- added link ring_tip
- added link thumb_tip
Joints:
- added joint index_joint_tip: type fixed, parent index_distal, child index_tip, origin xyz=0 0 0.026 rpy=0 0 0
- added joint little_joint_tip: type fixed, parent little_distal, child little_tip, origin xyz=0 0 0.026 rpy=0 0 0
- added joint middle_joint_tip: type fixed, parent middle_distal, child middle_tip, origin xyz=0 0 0.026 rpy=0 0 0
- added joint ring_joint_tip: type fixed, parent ring_distal, child ring_tip, origin xyz=0 0 0.026 rpy=0 0 0
- added joint thumb_joint_tip: type fixed, parent thumb_distal, child thumb_tip, origin xyz=0 0 0.028 rpy=0 0 0

File: src/assets/canonical_extended/urdf/allegro_hand_left.urdf (robot description, URDF)
Before this commit: robot DexterousHand, 24 links, 23 joints
Links:
- added link index_tip
- added link little_tip
- added link middle_tip
- added link ring_tip
- added link thumb_tip
Joints:
- added joint index_joint_tip: type fixed, parent index_distal, child index_tip, origin xyz=0 0 0.0387 rpy=0 0 0
- added joint little_joint_tip: type fixed, parent little_distal, child little_tip, origin xyz=0 0 0.0387 rpy=0 0 0
- added joint middle_joint_tip: type fixed, parent middle_distal, child middle_tip, origin xyz=0 0 0.0387 rpy=0 0 0
- added joint ring_joint_tip: type fixed, parent ring_distal, child ring_tip, origin xyz=0 0 0.0 rpy=0 0 0
- added joint thumb_joint_tip: type fixed, parent thumb_distal, child thumb_tip, origin xyz=0 0 0.0543 rpy=0 0 0

File: src/assets/canonical_extended/urdf/allegro_hand_right.urdf (robot description, URDF)
Before this commit: robot DexterousHand, 24 links, 23 joints
Links:
- added link index_tip
- added link little_tip
- added link middle_tip
- added link ring_tip
- added link thumb_tip
Joints:
- added joint index_joint_tip: type fixed, parent index_distal, child index_tip, origin xyz=0 0 0.0387 rpy=0 0 0
- added joint little_joint_tip: type fixed, parent little_distal, child little_tip, origin xyz=0 0 0.0387 rpy=0 0 0
- added joint middle_joint_tip: type fixed, parent middle_distal, child middle_tip, origin xyz=0 0 0.0387 rpy=0 0 0
- added joint ring_joint_tip: type fixed, parent ring_distal, child ring_tip, origin xyz=0 0 0.0 rpy=0 0 0
- added joint thumb_joint_tip: type fixed, parent thumb_distal, child thumb_tip, origin xyz=0 0 0.0543 rpy=0 0 0

File: src/assets/canonical_extended/urdf/barrett_hand.urdf (robot description, URDF)
Before this commit: robot DexterousHand, 24 links, 23 joints
Links:
- added link index_tip
- added link little_tip
- added link middle_tip
- added link ring_tip
- added link thumb_tip
Joints:
- added joint index_joint_tip: type fixed, parent index_distal, child index_tip, origin xyz=0 0 0.064 rpy=0 0 0
- added joint little_joint_tip: type fixed, parent little_distal, child little_tip, origin xyz=0 0 0.0 rpy=0 0 0
- added joint middle_joint_tip: type fixed, parent middle_distal, child middle_tip, origin xyz=0 0 0.064 rpy=0 0 0
- added joint ring_joint_tip: type fixed, parent ring_distal, child ring_tip, origin xyz=0 0 0.0 rpy=0 0 0
- added joint thumb_joint_tip: type fixed, parent thumb_distal, child thumb_tip, origin xyz=0 0 0.064 rpy=0 0 0

File: src/assets/canonical_extended/urdf/leap_hand_left.urdf (robot description, URDF)
Before this commit: robot DexterousHand, 24 links, 23 joints
Links:
- added link index_tip
- added link little_tip
- added link middle_tip
- added link ring_tip
- added link thumb_tip
Joints:
- added joint index_joint_tip: type fixed, parent index_distal, child index_tip, origin xyz=0 0 0.052 rpy=0 0 0
- added joint little_joint_tip: type fixed, parent little_distal, child little_tip, origin xyz=0 0 0.052 rpy=0 0 0
- added joint middle_joint_tip: type fixed, parent middle_distal, child middle_tip, origin xyz=0 0 0.052 rpy=0 0 0
- added joint ring_joint_tip: type fixed, parent ring_distal, child ring_tip, origin xyz=0 0 0.0 rpy=0 0 0
- added joint thumb_joint_tip: type fixed, parent thumb_distal, child thumb_tip, origin xyz=0 0 0.06 rpy=0 0 0

File: src/assets/canonical_extended/urdf/leap_hand_right.urdf (robot description, URDF)
Before this commit: robot DexterousHand, 24 links, 23 joints
Links:
- added link index_tip
- added link little_tip
- added link middle_tip
- added link ring_tip
- added link thumb_tip
Joints:
- added joint index_joint_tip: type fixed, parent index_distal, child index_tip, origin xyz=0 0 0.052 rpy=0 0 0
- added joint little_joint_tip: type fixed, parent little_distal, child little_tip, origin xyz=0 0 0.052 rpy=0 0 0
- added joint middle_joint_tip: type fixed, parent middle_distal, child middle_tip, origin xyz=0 0 0.052 rpy=0 0 0
- added joint ring_joint_tip: type fixed, parent ring_distal, child ring_tip, origin xyz=0 0 0.0 rpy=0 0 0
- added joint thumb_joint_tip: type fixed, parent thumb_distal, child thumb_tip, origin xyz=0 0 0.06 rpy=0 0 0

File: src/assets/canonical_extended/urdf/mano.urdf (robot description, URDF)
Before this commit: robot DexterousHand, 24 links, 23 joints
Links:
- added link index_tip
- added link little_tip
- added link middle_tip
- added link ring_tip
- added link thumb_tip
Joints:
- added joint index_joint_tip: type fixed, parent index_distal, child index_tip, origin xyz=0 0 0.0256 rpy=0 0 0
- added joint little_joint_tip: type fixed, parent little_distal, child little_tip, origin xyz=0 0 0.0189 rpy=0 0 0
- added joint middle_joint_tip: type fixed, parent middle_distal, child middle_tip, origin xyz=0 0 0.0243 rpy=0 0 0
- added joint ring_joint_tip: type fixed, parent ring_distal, child ring_tip, origin xyz=0 0 0.0248 rpy=0 0 0
- added joint thumb_joint_tip: type fixed, parent thumb_distal, child thumb_tip, origin xyz=0 0 0.0318 rpy=0 0 0

File: src/assets/canonical_extended/urdf/shadow_hand_left.urdf (robot description, URDF)
Before this commit: robot DexterousHand, 24 links, 23 joints
Links:
- added link index_tip
- added link little_tip
- added link middle_tip
- added link ring_tip
- added link thumb_tip
Joints:
- added joint index_joint_tip: type fixed, parent index_distal, child index_tip, origin xyz=0 0 0.035 rpy=0 0 0
- added joint little_joint_tip: type fixed, parent little_distal, child little_tip, origin xyz=0 0 0.035 rpy=0 0 0
- added joint middle_joint_tip: type fixed, parent middle_distal, child middle_tip, origin xyz=0 0 0.035 rpy=0 0 0
- added joint ring_joint_tip: type fixed, parent ring_distal, child ring_tip, origin xyz=0 0 0.035 rpy=0 0 0
- added joint thumb_joint_tip: type fixed, parent thumb_distal, child thumb_tip, origin xyz=0 0 0.035 rpy=0 0 0
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