Commit message: update assets for Sharpa Wave

File: src/assets/canonical/urdf/sharpa_wave_left.urdf (robot description, URDF)
Before this commit: robot DexterousHand, 29 links, 28 joints
Joints:
- joint thumb_joint3: limit lower=-0.5236 upper=1.3963 effort=1.0 velocity=1.0 -> lower=-0.3491 upper=0.3491 effort=1.0 velocity=1.0
- joint thumb_joint4: limit lower=-0.3491 upper=0.3491 effort=1.0 velocity=1.0 -> lower=-0.5236 upper=1.3963 effort=1.0 velocity=1.0
